File: UIs.kicad_sch (KiCad schematic)
At the start: 20 parts

Commit message: 定時
Parts:
- removed C11, C12, C3: 0.1u, Capacitor_SMD:C_0402_1005Metric_Pad0.74x0.62mm_HandSolder, symbol Device:C_Small
- removed RV1, RV10, RV9: R_Potentiometer_US, Potentiometer_THT:Potentiometer_Vishay_T73YP_Vertical, symbol Device:R_Potentiometer_US
Other:
- moved on the sheet: C10, C5, C6, C7, C8, C9, RV3, RV4, RV5, RV6, RV7, RV8
