File: jhl_synth3.kicad_pcb (KiCad board)
At the start: 2 copper layers, 127 parts, among them IC1 HTK16K33, J3 Conn_01x05, J4 DIN-5, J5 Conn_01x08, Q1 NPN 2N3904 SOT-23, Q2 NPN 2SC4116 SC-70, U1 YAAJ_WeAct_BlackPill_Part_Like, U2 TLP127, U6 PCA9306DP

Commit message: LED並べた、だけ。
Parts:
- moved D73 119.5 mm to (165.0, 103.0)
- moved D89 118.9 mm to (165.0, 106.8)
- moved D81 112.6 mm to (165.0, 112.5)
- moved D65 110.7 mm to (165.0, 104.9)
- moved D49 109.1 mm to (165.0, 97.4)
- moved D41 107.8 mm to (165.0, 110.6)
- moved D57 106.7 mm to (165.0, 114.3)
- moved D25 105.3 mm to (165.0, 101.2)
- moved D33 102.6 mm to (165.0, 118.1)
- moved D17 100.2 mm to (165.0, 108.7)
- moved D1 97.9 mm to (165.0, 99.3)
- moved D9 95.1 mm to (165.0, 116.2)
Changed lines of the file:
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@@
 	(footprint "LED_SMD:LED_0603_1608Metric_Pad1.05x0.95mm_HandSolder"
 		(layer "F.Cu")
-		(at 243.405 36.655)
+		(at 165.005 110.575455)
 		(descr "LED SMD 0603 (1608 Metric), square (rectangular) end terminal, IPC-7351 nominal, (Body size source: http://www.tortai-tech.com/upload/download/2011102023233369053.pdf)")
 		(tags "LED handsolder")
@@
 			(at 0 1.43 0)
 			(layer "F.Fab")
+			(hide yes)
 			(effects
 				(font
@@
 	(footprint "LED_SMD:LED_0603_1608Metric_Pad1.05x0.95mm_HandSolder"
 		(layer "F.Cu")
-		(at 247.8 26.295)
+		(at 165.005 97.39)
 		(descr "LED SMD 0603 (1608 Metric), square (rectangular) end terminal, IPC-7351 nominal, (Body size source: http://www.tortai-tech.com/upload/download/2011102023233369053.pdf)")
 		(tags "LED handsolder")
@@
 			(at 0 1.43 0)
 			(layer "F.Fab")
+			(hide yes)
 			(effects
 				(font
@@
 	(footprint "LED_SMD:LED_0603_1608Metric_Pad1.05x0.95mm_HandSolder"
 		(layer "F.Cu")
-		(at 234.615 36.655)
+		(at 165.005 108.691818)
 		(descr "LED SMD 0603 (1608 Metric), square (rectangular) end terminal, IPC-7351 nominal, (Body size source: http://www.tortai-tech.com/upload/download/2011102023233369053.pdf)")
 		(tags "LED handsolder")
@@
 			(at 0 1.43 0)
 			(layer "F.Fab")
+			(hide yes)
 			(effects
 				(font
@@
 	(footprint "LED_SMD:LED_0603_1608Metric_Pad1.05x0.95mm_HandSolder"
 		(layer "F.Cu")
-		(at 230.22 47.015)
+		(at 165.005 116.226364)
 		(descr "LED SMD 0603 (1608 Metric), square (rectangular) end terminal, IPC-7351 nominal, (Body size source: http://www.tortai-tech.com/upload/download/2011102023233369053.pdf)")
 		(tags "LED handsolder")
@@
 			(at 0 1.43 0)
 			(layer "F.Fab")
+			(hide yes)
 			(effects
 				(font
@@
 	(footprint "LED_SMD:LED_0603_1608Metric_Pad1.05x0.95mm_HandSolder"
 		(layer "F.Cu")
-		(at 247.8 47.015)
+		(at 165.005 114.342727)
 		(descr "LED SMD 0603 (1608 Metric), square (rectangular) end terminal, IPC-7351 nominal, (Body size source: http://www.tortai-tech.com/upload/download/2011102023233369053.pdf)")
 		(tags "LED handsolder")
@@
 			(at 0 1.43 0)
 			(layer "F.Fab")
+			(hide yes)
 			(effects
 				(font
@@
 	(footprint "LED_SMD:LED_0603_1608Metric_Pad1.05x0.95mm_HandSolder"
 		(layer "F.Cu")
-		(at 256.59 47.015)
+		(at 165.005 112.459091)
 		(descr "LED SMD 0603 (1608 Metric), square (rectangular) end terminal, IPC-7351 nominal, (Body size source: http://www.tortai-tech.com/upload/download/2011102023233369053.pdf)")
 		(tags "LED handsolder")
@@
 			(at 0 1.43 0)
 			(layer "F.Fab")
+			(hide yes)
 			(effects
 				(font
@@
 	(footprint "LED_SMD:LED_0603_1608Metric_Pad1.05x0.95mm_HandSolder"
 		(layer "F.Cu")
-		(at 252.195 36.655)
+		(at 165.005 104.924545)
 		(descr "LED SMD 0603 (1608 Metric), square (rectangular) end terminal, IPC-7351 nominal, (Body size source: http://www.tortai-tech.com/upload/download/2011102023233369053.pdf)")
 		(tags "LED handsolder")
@@
 			(at 0 1.43 0)
 			(layer "F.Fab")
+			(hide yes)
 			(effects
 				(font
@@
 	(footprint "LED_SMD:LED_0603_1608Metric_Pad1.05x0.95mm_HandSolder"
 		(layer "F.Cu")
-		(at 230.22 26.295)
+		(at 165.005 99.273636)
 		(descr "LED SMD 0603 (1608 Metric), square (rectangular) end terminal, IPC-7351 nominal, (Body size source: http://www.tortai-tech.com/upload/download/2011102023233369053.pdf)")
 		(tags "LED handsolder")
@@
 			(at 0 1.43 0)
 			(layer "F.Fab")
+			(hide yes)
 			(effects
 				(font
@@
 	(footprint "LED_SMD:LED_0603_1608Metric_Pad1.05x0.95mm_HandSolder"
 		(layer "F.Cu")
-		(at 239.01 47.015)
+		(at 165.005 118.11)
 		(descr "LED SMD 0603 (1608 Metric), square (rectangular) end terminal, IPC-7351 nominal, (Body size source: http://www.tortai-tech.com/upload/download/2011102023233369053.pdf)")
 		(tags "LED handsolder")
@@
 			(at 0 1.43 0)
 			(layer "F.Fab")
+			(hide yes)
 			(effects
 				(font
@@
 	(footprint "LED_SMD:LED_0603_1608Metric_Pad1.05x0.95mm_HandSolder"
 		(layer "F.Cu")
-		(at 239.01 26.295)
+		(at 165.005 101.157273)
 		(descr "LED SMD 0603 (1608 Metric), square (rectangular) end terminal, IPC-7351 nominal, (Body size source: http://www.tortai-tech.com/upload/download/2011102023233369053.pdf)")
 		(tags "LED handsolder")
@@
 			(at 0 1.43 0)
 			(layer "F.Fab")
+			(hide yes)
 			(effects
 				(font
@@
 	(footprint "LED_SMD:LED_0603_1608Metric_Pad1.05x0.95mm_HandSolder"
 		(layer "F.Cu")
-		(at 256.59 26.295)
+		(at 165.005 103.040909)
 		(descr "LED SMD 0603 (1608 Metric), square (rectangular) end terminal, IPC-7351 nominal, (Body size source: http://www.tortai-tech.com/upload/download/2011102023233369053.pdf)")
 		(tags "LED handsolder")
@@
 			(at 0 1.43 0)
 			(layer "F.Fab")
+			(hide yes)
 			(effects
 				(font
@@
 	(footprint "LED_SMD:LED_0603_1608Metric_Pad1.05x0.95mm_HandSolder"
 		(layer "F.Cu")
-		(at 260.985 36.655)
+		(at 165.005 106.808182)
 		(descr "LED SMD 0603 (1608 Metric), square (rectangular) end terminal, IPC-7351 nominal, (Body size source: http://www.tortai-tech.com/upload/download/2011102023233369053.pdf)")
 		(tags "LED handsolder")
@@
 			(at 0 1.43 0)
 			(layer "F.Fab")
+			(hide yes)
 			(effects
 				(font

Commit message: 日々更新
Other:
- board text added: "1.8 128x160 lcd"
- board text added: "monotronサイズ(筐体外形) 高さ：最厚で28mm 単四x2"
Changed lines of the file:
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@@
 		)
+	)
+	(gr_rect
+		(start 41.5 116.5)
+		(end 161.5 188.5)
+		(stroke
+			(width 0.1)
+			(type default)
+		)
+		(fill no)
+		(layer "Dwgs.User")
+	)
+	(gr_rect
+		(start 181 125)
+		(end 239 159.5)
+		(stroke
+			(width 0.1)
+			(type default)
+		)
+		(fill no)
+		(layer "Dwgs.User")
+	)
+	(gr_rect
+		(start 189.918851 128.01272)
+		(end 223.918851 157.01272)
+		(stroke
+			(width 0.1)
+			(type default)
+		)
+		(fill no)
+		(layer "Dwgs.User")
 	)
 	(gr_text "ピン配置よくよく\n確認すること！"
@@
 		)
 	)
+	(gr_text "monotronサイズ(筐体外形)\n高さ：最厚で28mm\n単四x2"
+		(at 143 194.5 0)
+		(layer "Dwgs.User")
+		(effects
+			(font
+				(size 1 1)
+				(thickness 0.15)
+			)
+			(justify left bottom)
+		)
+	)
+	(gr_text "1.8 128x160 lcd"
+		(at 201 133.5 0)
+		(layer "Dwgs.User")
+		(effects
+			(font
+				(size 1 1)
+				(thickness 0.15)
+			)
+			(justify left bottom)
+		)
+	)
+	(group ""
+		(members "80db0336-65de-408b-ae8c-dfd5e2860de6" "d105382f-2de8-46ca-b35e-36103415e8b9")
+	)
 	(embedded_fonts no)

Commit message: 定時
Parts:
- removed C11, C12, C3: 0.1u, Capacitor_SMD:C_0402_1005Metric_Pad0.74x0.62mm_HandSolder
- removed RV1, RV10, RV9: R_Potentiometer_US, Potentiometer_THT:Potentiometer_Vishay_T73YP_Vertical
- added D97: LED_Small_Filled, LED_SMD:LED_0603_1608Metric_Pad1.05x0.95mm_HandSolder, F.Cu at (161.2, 83.8)
- added D98: LED_Small_Filled, LED_SMD:LED_0603_1608Metric_Pad1.05x0.95mm_HandSolder, F.Cu at (161.2, 86.4)
- J3: value Conn_01x05 -> Conn_I2S
- J5: value Conn_01x08 -> Conn_LCD
- moved J5 134.6 mm to (107.5, 128.2)
- moved J4 125.9 mm to (119.5, 123.1), turned to -90 degrees
- moved RV8 124.3 mm to (49.6, 180.8), turned to -90 degrees
- moved RV7 119.1 mm to (50.0, 167.1), turned to -90 degrees
- moved RV6 113.6 mm to (50.0, 152.6), turned to -90 degrees
- moved U1 98.8 mm to (133.5, 119.8)
- moved RV3 77.3 mm to (69.1, 142.0)
- moved RV2 71.2 mm to (69.6, 127.5)
- moved RV5 70.7 mm to (50.0, 138.6), turned to -90 degrees
- moved RV4 66.9 mm to (49.5, 124.6), turned to -90 degrees
Connections:
- U1 pad 12: unconnected-(U1-PB4-Pad12) -> LCD_RESET
- U1 pad 16: unconnected-(U1-PB8-Pad16) -> sw2
- U1 pad 17: unconnected-(U1-PB9-Pad17) -> LCD_A0
- U1 pad 26: ADC0 -> sw1
- U1 pad 3: unconnected-(U1-PB14-Pad3) -> LED3
- U1 pad 35: ADC9 -> sw5
- U1 pad 36: unconnected-(U1-PB2-Pad36) -> sw4
- U1 pad 37: unconnected-(U1-PB10-Pad37) -> sw3
- U1 pad 5: unconnected-(U1-PA8-Pad5) -> LED2
Other:
- board text added: "monotronサイズ(筐体外形) 120 x 72 x 厚28mm 単四x2"
- board text added: "volca 筐体外形 193 x 115 x 厚46mm（含ツマミ） aria compact 188 x 106 x 37"
- board text removed: "monotronサイズ(筐体外形) 高さ：最厚で28mm 単四x2"
